File: adc_controller.kicad_sch (KiCad schematic)
At the start: 7 parts, among them J4 Conn_01x05

Commit message: Add files via upload
Parts:
- removed J4: Conn_01x05, symbol Connector_Generic:Conn_01x05
- added J3: Conn_01x06, symbol Connector_Generic:Conn_01x06
- C6: footprint (none) -> Capacitor_SMD:C_0805_2012Metric
- R_ADC1, R_ADC2, R_ADC3, R_ADC4: footprint (none) -> Resistor_SMD:R_0805_2012Metric
Connections:
- net GND: now also J3.5 (Pin_5), J3.6 (Pin_6)
- net at R_ADC2.2: now also J3.2 (Pin_2)
- net at R_ADC1.2: now also J3.1 (Pin_1)
- net at R_ADC3.2: now also J3.3 (Pin_3)
- net at R_ADC4.2: now also J3.4 (Pin_4)
Changed lines of the file:
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@@
 	(wire
 		(pts
-			(xy 238.76 130.81) (xy 246.38 130.81)
+			(xy 240.03 133.35) (xy 240.03 130.81)
 		)
 		(stroke
@@
 		)
 	)
+	(wire
+		(pts
+			(xy 240.03 130.81) (xy 246.38 130.81)
+		)
+		(stroke
+			(width 0)
+			(type default)
+		)
+	)
+	(wire
+		(pts
+			(xy 240.03 133.35) (xy 246.38 133.35)
+		)
+		(stroke
+			(width 0)
+			(type default)
+		)
+	)
 	(global_label "SCL_BUS"
 		(shape input)
@@
 	(global_label "GND"
 		(shape input)
-		(at 238.76 130.81 270)
+		(at 240.03 133.35 270)
 		(fields_autoplaced yes)
 		(effects
@@
 		)
 		(property "Intersheetrefs" "${INTERSHEET_REFS}"
-			(at 238.76 137.6657 90)
+			(at 240.03 140.2057 90)
 			(effects
 				(font
@@
 			)
 		)
-		(property "Footprint" ""
+		(property "Footprint" "Resistor_SMD:R_0805_2012Metric"
 			(at 242.57 124.968 90)
 			(effects
@@
 	)
 	(symbol
-		(lib_id "Connector_Generic:Conn_01x05")
+		(lib_id "Connector_Generic:Conn_01x06")
 		(at 251.46 125.73 0)
 		(unit 1)
@@
 		(dnp no)
 		(fields_autoplaced yes)
-		(property "Reference" "J4"
-			(at 254 124.4599 0)
+		(property "Reference" "J3"
+			(at 254 125.7299 0)
 			(effects
 				(font
@@
 			)
 		)
-		(property "Value" "Conn_01x05"
-			(at 254 126.9999 0)
+		(property "Value" "Conn_01x06"
+			(at 254 128.2699 0)
 			(effects
 				(font
@@
 			)
 		)
-		(property "Description" "Generic connector, single row, 01x05, script generated (kicad-library-utils/schlib/autogen/connector/)"
+		(property "Description" "Generic connector, single row, 01x06, script generated (kicad-library-utils/schlib/autogen/connector/)"
 			(at 251.46 125.73 0)
 			(effects
@@
 			)
 		)
+		(pin "2"
+		)
+		(pin "5"
+		)
 		(pin "1"
 		)
+		(pin "6"
+		)
+		(pin "4"
+		)
 		(pin "3"
-		)
-		(pin "2"
-		)
-		(pin "4"
-		)
-		(pin "5"
 		)
 		(instances
 			(project ""
 				(path "/c8d0e3cf-b697-430c-b4f3-c5285558b4ca/64b9c830-1dcb-42ca-8ce2-512d1a0b5a28"
-					(reference "J4")
+					(reference "J3")
 					(unit 1)
 				)
@@
 			)
 		)
-		(property "Footprint" ""
+		(property "Footprint" "Resistor_SMD:R_0805_2012Metric"
 			(at 242.57 127.508 90)
 			(effects
@@
 			)
 		)
-		(property "Footprint" ""
+		(property "Footprint" "Resistor_SMD:R_0805_2012Metric"
 			(at 242.57 122.428 90)
 			(effects
@@
 			)
 		)
-		(property "Footprint" ""
+		(property "Footprint" "Capacitor_SMD:C_0805_2012Metric"
 			(at 220.98 139.3952 0)
 			(effects
@@
 			)
 		)
-		(property "Footprint" ""
+		(property "Footprint" "Resistor_SMD:R_0805_2012Metric"
 			(at 242.57 130.048 90)
 			(effects

Commit message: Add files via upload
v1.2 : complete schematics with added footprints, PCB layout remaining
Parts:
- added C10, C7, C8, C9: 100nF, Capacitor_SMD:C_0805_2012Metric, symbol Device:C
- J3: footprint (none) -> Connector_PinSocket_2.54mm:PinSocket_1x06_P2.54mm_Vertical
Connections:
- net GND: now also C10.2, C7.1, C8.2, C9.1
- net at J3.2 (Pin_2), R_ADC2.2: now also C9.2
- net at U_ADC1.4 (AIN0): now also R_ADC4.2; no longer R_ADC4.1
- net at J3.1 (Pin_1), R_ADC1.2: now also C8.1
- net at J3.3 (Pin_3), R_ADC3.2: now also C10.1
- net at J3.4 (Pin_4): now also R_ADC4.1, C7.2; no longer R_ADC4.2
Other:
- note added: "ADC(max 3.3V input)"
- note removed: "max 3.3V input"
- moved on the sheet: J3, R_ADC1, R_ADC4

Commit message: Add files via upload
V5 : complete finish for v1, directly to-the-fab design.
Parts:
- C10, C6, C7, C8, C9: LCSC (none) -> C49678
- J3: LCSC (none) -> C40877
- R_ADC1, R_ADC2, R_ADC3: LCSC (none) -> C17513
- R_ADC4: value 1k -> 1K; LCSC (none) -> C17513
- U_ADC1: LCSC (none) -> C16581
Changed lines of the file:
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@@
+			)
+		)
+		(property "LCSC" "C17513"
+			(at 242.57 123.19 90)
+			(effects
+				(font
+					(size 1.27 1.27)
+				)
+				(hide yes)
 			)
 		)
@@
 			)
 		)
+		(property "LCSC" "C16581"
+			(at 228.6 125.73 90)
+			(effects
+				(font
+					(size 1.27 1.27)
+				)
+				(hide yes)
+			)
+		)
 		(pin "1"
 		)
@@
 			)
 		)
+		(property "LCSC" "C49678"
+			(at 242.57 116.84 0)
+			(effects
+				(font
+					(size 1.27 1.27)
+				)
+				(hide yes)
+			)
+		)
 		(pin "1"
 		)
@@
 			)
 		)
+		(property "LCSC" "C40877"
+			(at 257.81 125.73 0)
+			(effects
+				(font
+					(size 1.27 1.27)
+				)
+				(hide yes)
+			)
+		)
 		(pin "2"
 		)
@@
 			)
 		)
+		(property "LCSC" "C49678"
+			(at 247.65 119.38 0)
+			(effects
+				(font
+					(size 1.27 1.27)
+				)
+				(hide yes)
+			)
+		)
 		(pin "1"
 		)
@@
 			)
 		)
+		(property "LCSC" "C49678"
+			(at 242.57 132.08 0)
+			(effects
+				(font
+					(size 1.27 1.27)
+				)
+				(hide yes)
+			)
+		)
 		(pin "2"
 		)
@@
 			)
 		)
+		(property "LCSC" "C17513"
+			(at 242.57 125.73 90)
+			(effects
+				(font
+					(size 1.27 1.27)
+				)
+				(hide yes)
+			)
+		)
 		(pin "1"
 		)
@@
 			)
 		)
+		(property "LCSC" "C17513"
+			(at 238.76 116.84 0)
+			(effects
+				(font
+					(size 1.27 1.27)
+				)
+				(hide yes)
+			)
+		)
 		(pin "1"
 		)
@@
 			)
 		)
+		(property "LCSC" "C49678"
+			(at 247.65 129.54 0)
+			(effects
+				(font
+					(size 1.27 1.27)
+				)
+				(hide yes)
+			)
+		)
 		(pin "2"
 		)
@@
 			)
 		)
+		(property "LCSC" "C49678"
+			(at 224.79 138.43 0)
+			(effects
+				(font
+					(size 1.27 1.27)
+				)
+				(hide yes)
+			)
+		)
 		(pin "2"
 		)
@@
 			)
 		)
-		(property "Value" "1k"
+		(property "Value" "1K"
 			(at 241.3 133.3499 0)
 			(effects
@@
 			(at 238.76 132.08 0)
 			(effects
+				(font
+					(size 1.27 1.27)
+				)
+				(hide yes)
+			)
+		)
+		(property "LCSC" "C17513"
+			(at 238.76 132.08 0)
+			(effects
