File: pwm.kicad_sch (KiCad schematic)
At the start: 5 parts, among them J4 Conn_01x08, J6 Conn_01x04

Commit message: Add files via upload
v1.2 : complete schematics with added footprints, PCB layout remaining
Parts:
- J4: footprint (none) -> Connector_PinSocket_2.54mm:PinSocket_1x08_P2.54mm_Vertical
- J6: footprint (none) -> Connector_PinSocket_2.54mm:PinSocket_1x04_P2.54mm_Vertical
Changed lines of the file:
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@@
 			)
 		)
-		(property "Footprint" ""
+		(property "Footprint" "Connector_PinSocket_2.54mm:PinSocket_1x04_P2.54mm_Vertical"
 			(at 269.24 63.5 0)
 			(effects
@@
 			)
 		)
-		(property "Footprint" ""
+		(property "Footprint" "Connector_PinSocket_2.54mm:PinSocket_1x08_P2.54mm_Vertical"
 			(at 269.24 46.99 0)
 			(effects

Commit message: Add files via upload
V5 : complete finish for v1, directly to-the-fab design.
Parts:
- C5: LCSC (none) -> C49678
- J4: LCSC (none) -> C18078131
- J6: LCSC (none) -> C5116530
- R9: LCSC (none) -> C17414
- U_PWM1: LCSC (none) -> C11628
Changed lines of the file:
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@@
+			)
+		)
+		(property "LCSC" "C5116530"
+			(at 269.24 63.5 0)
+			(effects
+				(font
+					(size 1.27 1.27)
+				)
+				(hide yes)
 			)
 		)
@@
 			)
 		)
+		(property "LCSC" "C11628"
+			(at 238.76 57.15 0)
+			(effects
+				(font
+					(size 1.27 1.27)
+				)
+				(hide yes)
+			)
+		)
 		(pin "25"
 		)
@@
 			)
 		)
+		(property "LCSC" "C49678"
+			(at 242.57 31.75 90)
+			(effects
+				(font
+					(size 1.27 1.27)
+				)
+				(hide yes)
+			)
+		)
 		(pin "1"
 		)
@@
 			)
 		)
+		(property "LCSC" "C17414"
+			(at 219.71 50.8 0)
+			(effects
+				(font
+					(size 1.27 1.27)
+				)
+				(hide yes)
+			)
+		)
 		(pin "2"
 		)
@@
 			(at 269.24 46.99 0)
 			(effects
+				(font
+					(size 1.27 1.27)
+				)
+				(hide yes)
+			)
+		)
+		(property "LCSC" "C18078131"
+			(at 269.24 46.99 0)
+			(effects
